File: Electrical/Board Circuit/Board Circuit.sch (KiCad schematic (older format))
At the start: 26 parts

Commit message: Diddeli did some updating of the schematic and made some footprints
Parts:
- removed J?: Conn_01x05_Female, symbol Connector:Conn_01x05_Female
- removed Q? (x2): Q_PMOS_DGS, symbol Device:Q_PMOS_DGS
- removed Q? (x2): Q_NMOS_DGS, symbol Device:Q_NMOS_DGS
- removed Q? (x2): Q_NPN_BCE, symbol Device:Q_NPN_BCE
- removed U? (x5): 4081, symbol 4xxx:4081
- removed U? (x3): 4011, symbol 4xxx:4011
- added J1: Conn_01x06_Female, Connector_Wuerth:Wuerth_WR-WTB_64800611622_1x06_P1.50mm_Vertical, symbol Connector:Conn_01x06_Female
- added Q1, Q4: Q_PMOS_GDS, Board Circuit:PMOS, symbol Device:Q_PMOS_GDS
- added Q11, Q41: Q_NPN_CBE, Board Circuit:NPN CBE, symbol Device:Q_NPN_CBE
- added Q2, Q3: Q_NMOS_GDS, Board Circuit:PMOS, symbol Device:Q_NMOS_GDS
- added R13, R21, R31, R43: R, Resistor_THT:R_Axial_DIN0207_L6.3mm_D2.5mm_P10.16mm_Horizontal, symbol Device:R
- added U1: SN74HC08, Board Circuit:SN74HC08 AND, symbol Board~Circuit:SN74HC08
- added U2: SN74HCT00, Board Circuit:SN74HCT00 NAND, symbol Board~Circuit:SN74HCT00
- D1, D2: renamed from D?; footprint (none) -> Diode_THT:D_5KPW_P12.70mm_Horizontal
- L1: renamed from L?; footprint (none) -> Inductor_THT:L_Axial_L5.3mm_D2.2mm_P2.54mm_Vertical_Vishay_IM-1
- R11, R12, R14, R22, R32, R41, R42, R44: renamed from R?; footprint (none) -> Resistor_THT:R_Axial_DIN0207_L6.3mm_D2.5mm_P10.16mm_Horizontal
Connections:
- wire segments 79 -> 91
- no-connect marks 0 -> 1
Other:
- moved on the sheet: R22, R32, R44
